Commit message: test ok

File: urdf/udacity_bot.xacro (robot description, xacro)
@@ -146,4 +146,27 @@
     </visual>
   </link>
+  <link name='hokuyo'>
+    <inertial>
+      <mass value="0.1"/>
+      <origin xyz="0 0 0" rpy=" 0 0 0"/>
+      <inertia
+          ixx="1e-6" ixy="0" ixz="0"
+          iyy="1e-6" iyz="0"
+          izz="1e-6"
+      />
+    </inertial>
+    <collision name='hokuyo_collision'>
+      <origin xyz="0 0 0" rpy=" 0 0 0"/>
+      <geometry>
+        <box size="0.1 0.1 0.1"/>
+      </geometry>
+    </collision>
+    <visual name='hokuyo_visual'>
+      <origin xyz="0 0 0" rpy=" 0 0 0"/>
+      <geometry>
+        <mesh filename="package://slam_project/meshes/hokuyo.dae"/>
+      </geometry>
+    </visual>
+  </link>
   <joint type="continuous" name="left_wheel_hinge">
     <origin xyz="0 0.15 0" rpy="0 0 0"/>
@@ -165,4 +188,11 @@
     <origin xyz="0.15 0 0.1" rpy="0 0 1.5708"/>
     <child link="camera"/>
+    <parent link="chassis"/>
+    <limit effort="10000" velocity="1000"/>
+    <joint_properties damping="1.0" friction="1.0"/>
+  </joint>
+  <joint type="fixed" name="hokuyo_joint">
+    <origin xyz="0.15 0 0.1" rpy="0 0 0"/>
+    <child link="hokuyo"/>
     <parent link="chassis"/>
     <limit effort="10000" velocity="1000"/>

Commit message: camera location fixed

File: urdf/udacity_bot.xacro (robot description, xacro)
@@ -134,5 +134,5 @@
     </inertial>
     <collision name='camera_collision'>
-      <origin xyz="0 0 0" rpy="0 0 0"/>
+      <origin xyz="0 0 0" rpy="0 0 1.5707"/>
       <geometry>
         <box size="0.0730 .2760 0.0720"/>
@@ -140,5 +140,5 @@
     </collision>
     <visual name='camera_visual'>
-      <origin xyz="0 0 -0.02" rpy="0 0 0"/>
+      <origin xyz="0 0 -0.02" rpy="0 0 1.5707"/>
       <geometry>
         <mesh filename="package://slam_project/meshes/kinetic.dae"/>
@@ -186,5 +186,5 @@
   </joint>
   <joint type="fixed" name="camera_joint">
-    <origin xyz="0.15 0 0.1" rpy="0 0 1.5708"/>
+    <origin xyz="0.15 0 0.1" rpy="0 0 0"/>
     <child link="camera"/>
     <parent link="chassis"/>
@@ -215,4 +215,5 @@
   <joint name="camera_depth_optical_joint" type="fixed">
     <origin xyz="0 0 0" rpy="${-M_PI/2} 0 ${-M_PI/2}" />
+    <!-- <origin xyz="0 0 0" rpy="0 0 0" /> -->
     <parent link="camera_depth_frame" />
     <child link="camera_depth_optical_frame" />
@@ -243,4 +244,5 @@
   <joint name="camera_rgb_optical_joint" type="fixed">
     <origin xyz="0 0 0" rpy="${-M_PI/2} 0 ${-M_PI/2}" />
+    <!-- <origin xyz="0 0 0" rpy="0 0 0" /> -->
     <parent link="camera_rgb_frame" />
     <child link="camera_rgb_optical_frame" />
